File: output/pcbs/tutorial.kicad_pcb (KiCad board)
At the start: 2 copper layers, 266.3 x 131.4 mm, 127 parts

Commit message: 15 Apr 2025/04
Parts:
- moved D28 19.6 mm to (136.8, 181.7)
- moved S28 19.6 mm to (139.6, 177.6)
- moved D53 19.6 mm to (216.8, 163.7)
- moved S40 19.6 mm to (259.2, 122.2)
- moved D9 19.6 mm to (86.8, 158.9)
- moved D44 19.6 mm to (249.0, 146.7)
- moved D8 19.6 mm to (91.5, 93.5)
- moved D55 19.6 mm to (205.2, 131.8)
- moved S4 19.6 mm to (76.3, 82.7)
- moved S25 19.6 mm to (150.1, 143.1)
- moved OLED1 19.6 mm to (173.7, 162.1)
- moved D5 19.6 mm to (74.0, 141.5)
- moved D34 19.6 mm to (285.4, 141.5)
- moved D38 19.6 mm to (272.5, 158.9)
- moved S27 19.6 mm to (161.7, 111.1)
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Routing:
- net P14: track 0.00 -> 456.7 mm
- net P16: track 0.00 -> 433.2 mm
- net P10: track 0.00 -> 395.7 mm
- net P7: track 0.00 -> 363.4 mm
- net P8: track 0.00 -> 332.7 mm
- net P9: track 0.00 -> 272.5 mm
- net P18: track 0.00 -> 116.0 mm
- net P0: track 0.00 -> 113.4 mm
- net P1: track 0.00 -> 113.2 mm
- net P21: track 0.00 -> 113.0 mm
- net P19: track 0.00 -> 112.8 mm
- net P4: track 0.00 -> 112.4 mm
- net P20: track 0.00 -> 112.3 mm
- net P5: track 0.00 -> 108.5 mm
- net P6: track 0.00 -> 107.0 mm
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Other:
- net class Default removed

Commit message: 16 Apr 2025/01
Parts:
- moved D14 7.84 mm to (111.9, 165.6)
- moved S10 7.84 mm to (101.7, 141.1)
- moved S49 7.84 mm to (238.5, 153.4)
- moved S1 7.84 mm to (66.1, 133.5)
- moved D29 7.84 mm to (168.9, 195.5)
- moved S41 7.84 mm to (260.7, 109.1)
- moved D22 7.84 mm to (145.4, 126.2)
- moved D31 7.84 mm to (303.8, 122.2)
- moved D37 7.84 mm to (275.2, 96.4)
- moved D4 7.84 mm to (81.8, 90.2)
- moved D12 7.84 mm to (111.6, 113.8)
- moved S26 7.84 mm to (163.2, 130.0)
- moved S56 7.84 mm to (205.0, 114.0)
- moved S2 7.84 mm to (71.9, 117.5)
- moved D55 7.84 mm to (212.5, 134.7)
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Routing:
- net P14: track 456.7 -> 613.1 mm, vias 0 -> 1
- net P16: track 433.2 -> 573.9 mm, vias 0 -> 1
- net P10: track 395.7 -> 513.5 mm, vias 0 -> 1
- net P7: track 363.4 -> 454.5 mm, vias 0 -> 1
- net P8: track 332.7 -> 404.2 mm, vias 0 -> 1
- net P9: track 272.5 -> 339.7 mm, vias 0 -> 1
- net P15: track 103.7 -> 166.1 mm
- net P6: track 107.0 -> 164.3 mm
- net GND: track 0.00 -> 55.1 mm
- net P18: track 116.0 -> 170.9 mm
- net P5: track 108.5 -> 161.4 mm
- net P21: track 113.0 -> 157.8 mm
- net P19: track 112.8 -> 154.9 mm
- net RST: track 0.00 -> 38.8 mm
- net P20: track 112.3 -> 149.1 mm
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